File: Longan V2/Longan V2/Longan V2.kicad_sch (KiCad schematic)
At the start: 17 parts, among them J1 Conn_Coaxial, J2 Conn_Coaxial, J3 Conn_02x09_Odd_Even, J5 Battery, J6 Serial Output, SW1 Reset SW, U1 Ai-Thinker-Ra-01, U2 MAX-M8Q, U3 Pico

Commit message: Polishing
- More vias
- Test points
- Narrower zones
- Logo
- Pin Labels
Parts:
- added TP1: GPS_RX, TestPoint:TestPoint_Pad_D2.5mm, symbol Connector:TestPoint
- added TP2: GPS_TX, TestPoint:TestPoint_Pad_D2.5mm, symbol Connector:TestPoint
- added TP3, TP7: GND, TestPoint:TestPoint_Pad_D2.5mm, symbol Connector:TestPoint
- added TP4: Bat, TestPoint:TestPoint_Pad_D2.5mm, symbol Connector:TestPoint
- added TP5: 3v3, TestPoint:TestPoint_Pad_D2.5mm, symbol Connector:TestPoint
- added TP6: GNDA, TestPoint:TestPoint_Pad_D2.5mm, symbol Connector:TestPoint
Connections:
- net +3V3: now also TP5.1
- net BAT_IN: now also TP4.1
- net GND: now also TP3.1, TP7.1
- net GNDA: now also TP6.1
- net RX_1: now also TP1.1
- net TX_1: now also TP2.1
Other:
- title: Longan Main Board -> Longan Flight Computer
Changed lines of the file:
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@@
   (paper "A4")
   (title_block
-    (title "Longan Main Board")
+    (title "Longan Flight Computer")
     (date "2022-11-19")
     (rev "V2")
     (company "CUSF")
   )
+  (junction (at 190.5 49.53) (diameter 0) (color 0 0 0 0)
+  )
   (junction (at 114.3 69.85) (diameter 0) (color 0 0 0 0)
   )
@@
   (junction (at 233.68 114.3) (diameter 0) (color 0 0 0 0)
   )
+  (junction (at 114.3 44.45) (diameter 0) (color 0 0 0 0)
+  )
   (junction (at 78.74 151.13) (diameter 0) (color 0 0 0 0)
   )
+  (junction (at 190.5 57.15) (diameter 0) (color 0 0 0 0)
+  )
   (junction (at 45.72 40.64) (diameter 0) (color 0 0 0 0)
   )
@@
   (junction (at 52.07 40.64) (diameter 0) (color 0 0 0 0)
   )
+  (junction (at 31.75 140.97) (diameter 0) (color 0 0 0 0)
+  )
   (junction (at 114.3 82.55) (diameter 0) (color 0 0 0 0)
   )
   (junction (at 67.31 114.3) (diameter 0) (color 0 0 0 0)
+  )
+  (junction (at 29.21 143.51) (diameter 0) (color 0 0 0 0)
   )
   (junction (at 80.01 121.92) (diameter 0) (color 0 0 0 0)
@@
     (stroke (width 0) (type default) (color 0 0 0 0))
   )
+  (wire (pts (xy 190.5 57.15) (xy 196.85 57.15))
+    (stroke (width 0) (type default) (color 0 0 0 0))
+  )
   (wire (pts (xy 182.88 69.85) (xy 182.88 82.55))
     (stroke (width 0) (type default) (color 0 0 0 0))
@@
     (stroke (width 0) (type default) (color 0 0 0 0))
   )
+  (wire (pts (xy 190.5 49.53) (xy 196.85 49.53))
+    (stroke (width 0) (type default) (color 0 0 0 0))
+  )
   (polyline (pts (xy 91.44 97.79) (xy 91.44 20.32))
     (stroke (width 0) (type default) (color 0 0 0 0))
@@
     (stroke (width 0) (type default) (color 0 0 0 0))
   )
+  (wire (pts (xy 109.22 44.45) (xy 114.3 44.45))
+    (stroke (width 0) (type default) (color 0 0 0 0))
+  )
   (wire (pts (xy 78.74 151.13) (xy 81.28 151.13))
     (stroke (width 0) (type default) (color 0 0 0 0))
@@
     (stroke (width 0) (type default) (color 0 0 0 0))
   )
-  (wire (pts (xy 22.86 143.51) (xy 31.75 143.51))
+  (wire (pts (xy 22.86 143.51) (xy 29.21 143.51))
     (stroke (width 0) (type default) (color 0 0 0 0))
   )
@@
     (stroke (width 0) (type default) (color 0 0 0 0))
   )
+  (wire (pts (xy 29.21 128.27) (xy 29.21 143.51))
+    (stroke (width 0) (type default) (color 0 0 0 0))
+  )
   (wire (pts (xy 233.68 111.76) (xy 233.68 114.3))
     (stroke (width 0) (type default) (color 0 0 0 0))
@@
     (stroke (width 0) (type default) (color 0 0 0 0))
   )
-  (wire (pts (xy 176.53 41.91) (xy 166.37 41.91))
+  (wire (pts (xy 182.88 41.91) (xy 166.37 41.91))
     (stroke (width 0) (type default) (color 0 0 0 0))
   )
@@
     (stroke (width 0) (type default) (color 0 0 0 0))
   )
+  (wire (pts (xy 31.75 128.27) (xy 31.75 140.97))
+    (stroke (width 0) (type default) (color 0 0 0 0))
+  )
   (wire (pts (xy 245.11 55.88) (xy 245.11 52.07))
     (stroke (width 0) (type default) (color 0 0 0 0))
@@
   )
   (wire (pts (xy 55.88 58.42) (xy 64.77 58.42))
+    (stroke (width 0) (type default) (color 0 0 0 0))
+  )
+  (wire (pts (xy 29.21 143.51) (xy 31.75 143.51))
     (stroke (width 0) (type default) (color 0 0 0 0))
   )
@@
     )
     (property "Datasheet" "" (id 3) (at 80.01 123.19 0)
+      (effects (font (size 1.27 1.27)) hide)
+    )
+    (pin "1")
+  )
+  (symbol (lib_id "Connector:TestPoint") (at 196.85 49.53 0) (unit 1)
+    (in_bom yes) (on_board yes)
+    (property "Reference" "TP5" (id 0) (at 199.39 45.72 0)
+      (effects (font (size 1.27 1.27)) (justify left))
+    )
+    (property "Value" "3v3" (id 1) (at 199.39 48.26 0)
+      (effects (font (size 1.27 1.27)) (justify left))
+    )
+    (property "Footprint" "TestPoint:TestPoint_Pad_D2.5mm" (id 2) (at 201.93 49.53 0)
+      (effects (font (size 1.27 1.27)) hide)
+    )
+    (property "Datasheet" "~" (id 3) (at 201.93 49.53 0)
       (effects (font (size 1.27 1.27)) hide)
     )
@@
     )
     (property "Datasheet" "" (id 3) (at 45.72 86.36 0)
+      (effects (font (size 1.27 1.27)) hide)
+    )
+    (pin "1")
+  )
+  (symbol (lib_id "Connector:TestPoint") (at 31.75 128.27 0) (unit 1)
+    (in_bom yes) (on_board yes)
+    (property "Reference" "TP2" (id 0) (at 34.29 124.46 0)
+      (effects (font (size 1.27 1.27)) (justify left))
+    )
+    (property "Value" "GPS_TX" (id 1) (at 34.29 127 0)
+      (effects (font (size 1.27 1.27)) (justify left))
+    )
+    (property "Footprint" "TestPoint:TestPoint_Pad_D2.5mm" (id 2) (at 36.83 128.27 0)
+      (effects (font (size 1.27 1.27)) hide)
+    )
+    (property "Datasheet" "~" (id 3) (at 36.83 128.27 0)
+      (effects (font (size 1.27 1.27)) hide)
+    )
+    (pin "1")
+  )
+  (symbol (lib_id "Connector:TestPoint") (at 196.85 57.15 0) (unit 1)
+    (in_bom yes) (on_board yes)
+    (property "Reference" "TP6" (id 0) (at 199.39 53.34 0)
+      (effects (font (size 1.27 1.27)) (justify left))
+    )
+    (property "Value" "GNDA" (id 1) (at 199.39 55.88 0)
+      (effects (font (size 1.27 1.27)) (justify left))
+    )
+    (property "Footprint" "TestPoint:TestPoint_Pad_D2.5mm" (id 2) (at 201.93 57.15 0)
+      (effects (font (size 1.27 1.27)) hide)
+    )
+    (property "Datasheet" "~" (id 3) (at 201.93 57.15 0)
       (effects (font (size 1.27 1.27)) hide)
     )
@@
     (pin "9")
   )
+  (symbol (lib_id "Connector:TestPoint") (at 109.22 44.45 0) (unit 1)
+    (in_bom yes) (on_board yes)
+    (property "Reference" "TP3" (id 0) (at 106.68 35.56 0)
+      (effects (font (size 1.27 1.27)) (justify left))
+    )
+    (property "Value" "GND" (id 1) (at 106.68 38.1 0)
+      (effects (font (size 1.27 1.27)) (justify left))
+    )
+    (property "Footprint" "TestPoint:TestPoint_Pad_D2.5mm" (id 2) (at 114.3 44.45 0)
+      (effects (font (size 1.27 1.27)) hide)
+    )
+    (property "Datasheet" "~" (id 3) (at 114.3 44.45 0)
+      (effects (font (size 1.27 1.27)) hide)
+    )
+    (pin "1")
+  )
   (symbol (lib_id "Device:L") (at 78.74 137.16 0) (unit 1)
     (in_bom yes) (on_board yes) (fields_autoplaced)
@@
   )
   (symbol (lib_id "power:+3V3") (at 190.5 48.26 0) (unit 1)
-    (in_bom yes) (on_board yes) (fields_autoplaced)
+    (in_bom yes) (on_board yes)
     (property "Reference" "#PWR0105" (id 0) (at 190.5 52.07 0)
       (effects (font (size 1.27 1.27)) hide)
@@
     (pin "1")
   )
+  (symbol (lib_id "Connector:TestPoint") (at 114.3 44.45 0) (unit 1)
+    (in_bom yes) (on_board yes)
+    (property "Reference" "TP7" (id 0) (at 111.76 35.56 0)
+      (effects (font (size 1.27 1.27)) (justify left))
+    )
+    (property "Value" "GND" (id 1) (at 111.76 38.1 0)
+      (effects (font (size 1.27 1.27)) (justify left))
+    )
+    (property "Footprint" "TestPoint:TestPoint_Pad_D2.5mm" (id 2) (at 119.38 44.45 0)
+      (effects (font (size 1.27 1.27)) hide)
+    )
+    (property "Datasheet" "~" (id 3) (at 119.38 44.45 0)
+      (effects (font (size 1.27 1.27)) hide)
+    )
+    (pin "1")
+  )
   (symbol (lib_id "Device:C") (at 52.07 44.45 180) (unit 1)
     (in_bom yes) (on_board yes) (fields_autoplaced)
@@
     )
     (property "Datasheet" "" (id 3) (at 45.72 36.83 0)
+      (effects (font (size 1.27 1.27)) hide)
+    )
+    (pin "1")
+  )
+  (symbol (lib_id "Connector:TestPoint") (at 29.21 128.27 0) (unit 1)
+    (in_bom yes) (on_board yes)
+    (property "Reference" "TP1" (id 0) (at 24.13 124.46 0)
+      (effects (font (size 1.27 1.27)) (justify left))
+    )
+    (property "Value" "GPS_RX" (id 1) (at 20.32 127 0)
+      (effects (font (size 1.27 1.27)) (justify left))
+    )
+    (property "Footprint" "TestPoint:TestPoint_Pad_D2.5mm" (id 2) (at 34.29 128.27 0)
+      (effects (font (size 1.27 1.27)) hide)
+    )
+    (property "Datasheet" "~" (id 3) (at 34.29 128.27 0)
+      (effects (font (size 1.27 1.27)) hide)
+    )
+    (pin "1")
+  )
+  (symbol (lib_id "Connector:TestPoint") (at 182.88 41.91 0) (unit 1)
+    (in_bom yes) (on_board yes)
+    (property "Reference" "TP4" (id 0) (at 185.42 35.56 0)
+      (effects (font (size 1.27 1.27)) (justify left))
+    )
+    (property "Value" "Bat" (id 1) (at 185.42 38.1 0)
+      (effects (font (size 1.27 1.27)) (justify left))
+    )
+    (property "Footprint" "TestPoint:TestPoint_Pad_D2.5mm" (id 2) (at 187.96 41.91 0)
+      (effects (font (size 1.27 1.27)) hide)
+    )
+    (property "Datasheet" "~" (id 3) (at 187.96 41.91 0)
       (effects (font (size 1.27 1.27)) hide)
     )
@@
       (reference "SW1") (unit 1) (value "Reset SW") (footprint "Button_Switch_SMD:SW_Push_1P1T_NO_CK_KMR2")
     )
+    (path "/ed60b656-38c6-4ff0-9a1a-2d9003021990"
+      (reference "TP1") (unit 1) (value "GPS_RX") (footprint "TestPoint:TestPoint_Pad_D2.5mm")
+    )
+    (path "/6e04fb89-61d0-4a40-95b3-8b7efb404f18"
+      (reference "TP2") (unit 1) (value "GPS_TX") (footprint "TestPoint:TestPoint_Pad_D2.5mm")
+    )
+    (path "/7ab0c239-9378-40eb-b92b-83336ba6ead4"
+      (reference "TP3") (unit 1) (value "GND") (footprint "TestPoint:TestPoint_Pad_D2.5mm")
+    )
+    (path "/ff0a1273-c867-4abd-8d21-0191b42e3430"
+      (reference "TP4") (unit 1) (value "Bat") (footprint "TestPoint:TestPoint_Pad_D2.5mm")
+    )
+    (path "/19722243-4102-4d59-a829-b887da3b799d"
+      (reference "TP5") (unit 1) (value "3v3") (footprint "TestPoint:TestPoint_Pad_D2.5mm")
+    )
+    (path "/71333751-7af7-4225-a440-bb30ae6262e0"
+      (reference "TP6") (unit 1) (value "GNDA") (footprint "TestPoint:TestPoint_Pad_D2.5mm")
+    )
+    (path "/dbfd03d8-aedf-4042-a33b-f196df532d23"
+      (reference "TP7") (unit 1) (value "GND") (footprint "TestPoint:TestPoint_Pad_D2.5mm")
+    )
     (path "/ccdf1f17-1c14-4145-96c1-ef8b7e81b056"
